File: Breadboard Power Supply.kicad_pcb (KiCad board)
At the start: 2 copper layers, 0 parts

Commit message: schematic + placing
Parts:
- added C1: 10u, Capacitor_THT:C_Disc_D3.0mm_W1.6mm_P2.50mm, F.Cu at (158.6, 51.6)
- added C2: 1u, Capacitor_THT:C_Disc_D3.0mm_W1.6mm_P2.50mm, F.Cu at (156.7, 89.8)
- added C3: 0.1u, Capacitor_THT:C_Disc_D3.0mm_W1.6mm_P2.50mm, F.Cu at (152.9, 51.6)
- added D1: LED, PCM_LED_THT_AKL:LED_D5.0mm, F.Cu at (171.6, 72.0)
- added J1: Conn_01x02, Connector_PinHeader_2.54mm:PinHeader_1x02_P2.54mm_Vertical, F.Cu at (179.2, 47.7)
- added J2: Conn_01x02, Connector_PinHeader_2.54mm:PinHeader_1x02_P2.54mm_Vertical, F.Cu at (179.2, 93.5)
- added J3: Conn_01x03, Connector_PinHeader_2.54mm:PinHeader_1x03_P2.54mm_Vertical, F.Cu at (154.0, 96.2)
- added J4: Screw_Terminal_01x02, TerminalBlock:TerminalBlock_bornier-2_P5.08mm, F.Cu at (166.3, 49.8)
- added J5: Barrel_Jack_Switch, Connector_BarrelJack:BarrelJack_Horizontal, F.Cu at (162.6, 70.6)
- added J6: Conn_01x03, Connector_PinHeader_2.54mm:PinHeader_1x03_P2.54mm_Vertical, F.Cu at (154.1, 47.5)
- added J7: Screw_Terminal_01x02, TerminalBlock:TerminalBlock_bornier-2_P5.08mm, F.Cu at (166.3, 94.0)
- added R1: 330, PCM_Resistor_THT_AKL:R_Axial_DIN0204_L3.6mm_D1.6mm_P7.62mm_Horizontal, F.Cu at (167.8, 65.2)
- added R2: 330, PCM_Resistor_THT_AKL:R_Axial_DIN0204_L3.6mm_D1.6mm_P7.62mm_Horizontal, F.Cu at (167.6, 79.1)
- added R3: 560, PCM_Resistor_THT_AKL:R_Axial_DIN0204_L3.6mm_D1.6mm_P7.62mm_Horizontal, F.Cu at (167.6, 82.2)
- added S1: EG1218, digikey-footprints:Switch_Slide_11.6x4mm_EG1218, F.Cu at (173.0, 60.7)
- added U1: LM7805_TO220, Package_TO_SOT_THT:TO-220-3_Vertical, F.Cu at (159.5, 57.7)
- added U2: LM317_TO-220, Package_TO_SOT_THT:TO-220-3_Vertical, F.Cu at (154.3, 83.1)
Other:
- board outline added: 35.8 x 53.8 mm
