File: Breadboard Power Supply.kicad_pcb (KiCad board)
At the start: 2 copper layers, 35.8 x 53.8 mm, 17 parts, among them J1 Conn_01x02, J2 Conn_01x02, J3 Conn_01x03, J4 Screw_Terminal_01x02, J5 Barrel_Jack_Switch, J6 Conn_01x03, J7 Screw_Terminal_01x02, U1 LM7805_TO220, U2 LM317_TO-220

Commit message: Update Breadboard Power Supply.kicad_pcb
Routing:
- net GND: track 0.00 -> 110.8 mm
- net /PWR_output: track 0.00 -> 93.5 mm
- net /3.3V: track 0.00 -> 78.8 mm
- net /12V: track 0.00 -> 55.2 mm
- net /5V: track 0.00 -> 51.1 mm
- net Net-(U2-ADJ): track 0.00 -> 38.2 mm
- net /PWR_input: track 0.00 -> 13.3 mm
- net Net-(D1-A): track 0.00 -> 6.20 mm
Other:
- board size 35.8 x 53.8 mm -> 34.2 x 54.4 mm
- board text added: "GND"

Commit message: fix short circuit pwr_output
Connections:
- J1 pad 1: /PWR_output -> /PWR_OUT_BOTTOM
- J2 pad 1: /PWR_output -> /PWR_OUT_TOP
- J3 pad 2: /PWR_output -> /PWR_OUT_BOTTOM
- J4 pad 1: /PWR_output -> /PWR_OUT_BOTTOM
- J6 pad 2: /PWR_output -> /PWR_OUT_TOP
- J7 pad 1: /PWR_output -> /PWR_OUT_TOP
Routing:
- net /PWR_output: track 93.5 -> 0.00 mm
- net /PWR_OUT_TOP: track 0.00 -> 80.8 mm, vias 0 -> 1
- net /PWR_OUT_BOTTOM: track 0.00 -> 67.9 mm
- net /3.3V: track 78.8 -> 81.0 mm
